File: classes/03_homework/schema/schema.kicad_sch (KiCad schematic)
At the start: 11 parts

Commit message: Upload task schema
Parts:
- removed R? (x8): R, symbol Device:R
- removed U?: 74164, symbol 74xx_IEEE:74164
- removed U?: HDSM-543B, Display:HDSM-541B_HDSM-543B, symbol Display_Character:HDSM-543B
- removed U?: STM32F042C6Ux, Package_DFN_QFN:QFN-48-1EP_7x7mm_P0.5mm_EP5.6x5.6mm, symbol MCU_ST_STM32F0:STM32F042C6Ux
- added Q?_(NPN) (x2): BC546, Package_TO_SOT_THT:TO-92_Inline, symbol Transistor_BJT:BC546
- added Q?_(PNP) (x2): BC327, Package_TO_SOT_THT:TO-92_Inline, symbol Transistor_BJT:BC327
- added R10k (x6), R470 (x8): R, symbol Device:R
- added U?: STM32F215RETx, Package_QFP:LQFP-64_10x10mm_P0.5mm, symbol MCU_ST_STM32F2:STM32F215RETx
- added U?: 74164, symbol 74xx_IEEE:74164
- added U?: HDSM-541B, Display:HDSM-441B_HDSM-443B, symbol Display_Character:HDSM-541B
Connections:
- net Vdd: now also U?.14 (Vdd)
- net Vss: now also U?.7 (Vss)
- new net: R470.1, U?.5 (Qc)
- new net: R470.2, U?.8 (C)
- new net: Q?_(PNP).2 (B), R10k.1, R10k.2 (x2)
- new net: Q?_(NPN).1 (C), R10k.2 (x2)
- new net: R470.1, U?.3 (Qa)
- new net: R470.2, U?.3 (A)
- new net: Q?_(NPN).2 (B), R10k.2 (x2)
- new net: R470.1, U?.6 (Qd)
- new net: R470.2, U?.6 (D)
- new net: R470.1, U?.10 (Qe)
- new net: R470.2, U?.7 (E)
- new net: R470.1, U?.12 (Qg)
- new net: R470.2, U?.1 (G)
- new net: R470.1, U?.4 (Qb)
- new net: R470.2, U?.9 (B)
- new net: R470.1, U?.11 (Qf)
- new net: R470.1, U?.13 (Qh)
- new net: R470.2, U?.2 (DP)
- new net: R470.2, U?.4 (F)
- new net A1 - LEFT LIGHT: Q?_(PNP).3 (E), U?.10 (CA_DIG1)
- new net A2 - RIGHT LIGHT: Q?_(PNP).3 (E), U?.5 (CA_DIG2)
- new net GNDD: Q?_(NPN).3 (E), Q?_(NPN).3 (E)
- new net PA11 - in|OK: U?.44 (PA11)
- new net PB5 - out|RESET: U?.57 (PB5), U?.9 (~{R})
- new net PB6 - out|CLK: U?.58 (PB6), U?.8 (CK)
- new net PB7 - out|DATA: U?.1 (A), U?.2 (B), U?.59 (PB7)
- new net PB8 - out|LEFT LIGHT: R10k.1, U?.61 (PB8)
- new net PB9 - out|RIGHT LIGHT: R10k.1, U?.62 (PB9)
- new net PC6 - in|UP: U?.37 (PC6)
- new net PC7 - in|DOWN: U?.38 (PC7)
- new net Up - 5V: Q?_(PNP).1 (C), Q?_(PNP).1 (C), R10k.1, R10k.1
Other:
- note added: "QA - A QB - B QC - C QD - D QE - E QF - F QG - G QH - DP"

Commit message: Fix spelling in schema
Connections:
- net A1 - LEFT LIGHT renamed LEFT LIGHT
- net A2 - RIGHT LIGHT renamed RIGHT LIGHT
Changed lines of the file:
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@@
     (effects (font (size 1.27 1.27)) (justify left bottom))
   )
-  (label "A2 - RIGHT LIGHT" (at 198.12 220.98 0)
+  (label "RIGHT LIGHT" (at 198.12 220.98 0)
     (effects (font (size 1.27 1.27)) (justify left bottom))
   )
@@
     (effects (font (size 1.27 1.27)) (justify left bottom))
   )
-  (label "A1 - LEFT LIGHT" (at 198.12 218.44 0)
+  (label "LEFT LIGHT" (at 198.12 218.44 0)
     (effects (font (size 1.27 1.27)) (justify left bottom))
   )

Commit message: Fix the circuit schema
Parts:
- added C?: C, symbol Device:C
Connections:
- net Vdd is gone; now on net GNDD: U?.14 (Vdd)
- net Vss is gone; now on net GNDD: U?.7 (Vss)
- net GNDD: now also Q?_(PNP).3 (E), Q?_(PNP).3 (E), R10k.1, R10k.1, C?.1, C?.2
- net LEFT LIGHT: now also Q?_(PNP).1 (C); no longer Q?_(PNP).3 (E)
- net RIGHT LIGHT: now also Q?_(PNP).1 (C); no longer Q?_(PNP).3 (E)
- removed net Up - 5V: Q?_(PNP).1 (C), Q?_(PNP).1 (C), R10k.1, R10k.1
Changed lines of the file:
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@@
   (junction (at 207.01 134.62) (diameter 0) (color 0 0 0 0)
   )
+  (junction (at 134.62 187.96) (diameter 0) (color 0 0 0 0)
+  )
   (junction (at 266.7 121.92) (diameter 0) (color 0 0 0 0)
   )
@@
   (junction (at 207.01 121.92) (diameter 0) (color 0 0 0 0)
   )
+  (junction (at 129.54 187.96) (diameter 0) (color 0 0 0 0)
+  )
   (junction (at 191.77 146.05) (diameter 0) (color 0 0 0 0)
   )
@@
   (junction (at 257.81 121.92) (diameter 0) (color 0 0 0 0)
   )
+  (bus_entry (at 220.98 132.08) (size 2.54 2.54)
+    (stroke (width 0) (type default) (color 0 0 0 0))
+  )
+  (bus_entry (at 213.36 134.62) (size 2.54 2.54)
+    (stroke (width 0) (type default) (color 0 0 0 0))
+  )
   (wire (pts (xy 207.01 121.92) (xy 215.9 121.92))
     (stroke (width 0) (type default) (color 0 0 0 0))
@@
     (stroke (width 0) (type default) (color 0 0 0 0))
   )
+  (wire (pts (xy 162.56 187.96) (xy 162.56 146.05))
+    (stroke (width 0) (type default) (color 0 0 0 0))
+  )
   (polyline (pts (xy 105.41 182.88) (xy 203.2 182.88))
     (stroke (width 0) (type default) (color 0 0 0 0))
@@
     (stroke (width 0) (type default) (color 0 0 0 0))
   )
+  (wire (pts (xy 128.27 187.96) (xy 128.27 184.15))
+    (stroke (width 0) (type default) (color 0 0 0 0))
+  )
   (wire (pts (xy 215.9 129.54) (xy 215.9 121.92))
     (stroke (width 0) (type default) (color 0 0 0 0))
   )
+  (wire (pts (xy 134.62 184.15) (xy 135.89 184.15))
+    (stroke (width 0) (type default) (color 0 0 0 0))
+  )
   (wire (pts (xy 115.57 205.74) (xy 110.49 205.74))
     (stroke (width 0) (type default) (color 0 0 0 0))
@@
     (stroke (width 0) (type default) (color 0 0 0 0))
   )
+  (wire (pts (xy 129.54 194.31) (xy 129.54 187.96))
+    (stroke (width 0) (type default) (color 0 0 0 0))
+  )
   (wire (pts (xy 97.79 176.53) (xy 97.79 203.2))
     (stroke (width 0) (type default) (color 0 0 0 0))
@@
     (stroke (width 0) (type default) (color 0 0 0 0))
   )
+  (wire (pts (xy 129.54 187.96) (xy 128.27 187.96))
+    (stroke (width 0) (type default) (color 0 0 0 0))
+  )
   (wire (pts (xy 257.81 121.92) (xy 266.7 121.92))
     (stroke (width 0) (type default) (color 0 0 0 0))
@@
     (stroke (width 0) (type default) (color 0 0 0 0))
   )
+  (wire (pts (xy 129.54 187.96) (xy 129.54 121.92))
+    (stroke (width 0) (type default) (color 0 0 0 0))
+  )
   (wire (pts (xy 100.33 179.07) (xy 125.73 179.07))
     (stroke (width 0) (type default) (color 0 0 0 0))
@@
     (stroke (width 0) (type default) (color 0 0 0 0))
   )
+  (wire (pts (xy 129.54 121.92) (xy 207.01 121.92))
+    (stroke (width 0) (type default) (color 0 0 0 0))
+  )
   (wire (pts (xy 191.77 144.78) (xy 191.77 146.05))
     (stroke (width 0) (type default) (color 0 0 0 0))
@@
     (stroke (width 0) (type default) (color 0 0 0 0))
   )
+  (wire (pts (xy 134.62 194.31) (xy 134.62 187.96))
+    (stroke (width 0) (type default) (color 0 0 0 0))
+  )
   (wire (pts (xy 151.13 218.44) (xy 157.48 218.44))
     (stroke (width 0) (type default) (color 0 0 0 0))
@@
     (stroke (width 0) (type default) (color 0 0 0 0))
   )
-  (wire (pts (xy 163.83 121.92) (xy 207.01 121.92))
-    (stroke (width 0) (type default) (color 0 0 0 0))
-  )
   (wire (pts (xy 242.57 134.62) (xy 246.38 134.62))
     (stroke (width 0) (type default) (color 0 0 0 0))
   )
+  (wire (pts (xy 129.54 187.96) (xy 134.62 187.96))
+    (stroke (width 0) (type default) (color 0 0 0 0))
+  )
   (wire (pts (xy 99.06 199.39) (xy 115.57 199.39))
     (stroke (width 0) (type default) (color 0 0 0 0))
@@
     (stroke (width 0) (type default) (color 0 0 0 0))
   )
+  (wire (pts (xy 134.62 187.96) (xy 162.56 187.96))
+    (stroke (width 0) (type default) (color 0 0 0 0))
+  )
   (wire (pts (xy 110.49 203.2) (xy 115.57 203.2))
     (stroke (width 0) (type default) (color 0 0 0 0))
   )
   (wire (pts (xy 242.57 144.78) (xy 242.57 146.05))
+    (stroke (width 0) (type default) (color 0 0 0 0))
+  )
+  (wire (pts (xy 134.62 187.96) (xy 134.62 184.15))
     (stroke (width 0) (type default) (color 0 0 0 0))
   )
@@
   (label "RIGHT LIGHT" (at 266.7 161.29 90)
     (effects (font (size 1.27 1.27)) (justify left bottom))
+  )
+  (symbol (lib_id "Device:C") (at 132.08 184.15 90) (unit 1)
+    (in_bom yes) (on_board yes) (fields_autoplaced)
+    (property "Reference" "C?" (id 0) (at 132.08 176.53 90))
+    (property "Value" "C" (id 1) (at 132.08 179.07 90))
+    (property "Footprint" "" (id 2) (at 135.89 183.1848 0)
+      (effects (font (size 1.27 1.27)) hide)
+    )
+    (property "Datasheet" "~" (id 3) (at 132.08 184.15 0)
+      (effects (font (size 1.27 1.27)) hide)
+    )
+    (pin "1")
+    (pin "2")
   )
   (symbol (lib_id "MCU_ST_STM32F2:STM32F215RETx") (at 74.93 69.85 0) (unit 1)
@@
     (pin "2")
   )
-  (symbol (lib_id "Transistor_BJT:BC327") (at 213.36 134.62 0) (unit 1)
+  (symbol (lib_id "Transistor_BJT:BC327") (at 213.36 134.62 0) (mirror x) (unit 1)
     (in_bom yes) (on_board yes) (fields_autoplaced)
     (property "Reference" "Q?_(PNP)" (id 0) (at 218.44 133.3499 0)
@@
       (effects (font (size 1.27 1.27)) (justify left))
     )
-    (property "Footprint" "Package_TO_SOT_THT:TO-92_Inline" (id 2) (at 218.44 136.525 0)
+    (property "Footprint" "Package_TO_SOT_THT:TO-92_Inline" (id 2) (at 218.44 132.715 0)
       (effects (font (size 1.27 1.27) italic) (justify left) hide)
     )
@@
     (pin "2")
   )
-  (symbol (lib_id "Transistor_BJT:BC327") (at 264.16 134.62 0) (unit 1)
+  (symbol (lib_id "Transistor_BJT:BC327") (at 264.16 134.62 0) (mirror x) (unit 1)
     (in_bom yes) (on_board yes) (fields_autoplaced)
     (property "Reference" "Q?_(PNP)" (id 0) (at 269.24 133.3499 0)
@@
       (effects (font (size 1.27 1.27)) (justify left))
     )
-    (property "Footprint" "Package_TO_SOT_THT:TO-92_Inline" (id 2) (at 269.24 136.525 0)
+    (property "Footprint" "Package_TO_SOT_THT:TO-92_Inline" (id 2) (at 269.24 132.715 0)
       (effects (font (size 1.27 1.27) italic) (justify left) hide)
     )
@@
       (reference "#PWR?") (unit 1) (value "GNDD") (footprint "")
     )
+    (path "/02ff8bc7-c4a4-4544-93e3-f884d252c69d"
+      (reference "C?") (unit 1) (value "C") (footprint "")
+    )
     (path "/57fffba5-30ca-4bf5-8df9-b73f79ffb3a1"
