File: classes/05_sber-dat/schema/sber-dat/sber-dat.kicad_sch (KiCad schematic)
At the start: 0 parts

Commit message: Design the circuid
Parts:
- added L?: INDUCTOR, symbol pspice:INDUCTOR
- added R? (x3): R, symbol Device:R
- added U?: STM32L100, symbol custom:STM32L100
- added U?: Opamp_Dual, symbol Device:Opamp_Dual
Connections:
- new net: L?.2, R?.1, U?.3 (+)
- new net: R?.1, R?.1, U?.2 (-)
- new net (PWM) TIM2_CH2: L?.1, U?.24 (PA1)
- new net ADC1_IN10: R?.2, U?.1, U?.15 (PC0)
- new net GND: R?.2, R?.2, U?. (VBAT)
- new net I2C2_SCL: U?.47 (PB10)
- new net I2C2_SDA: U?.48 (PB11)
- new net MISO: U?.31 (PA6)
- new net MOSI: U?.32 (PA7)
- new net NSS: U?.29 (PA4)
- new net RX: U?.26 (PA3)
- new net SCK: U?.30 (PA5)
- new net TX: U?.25 (PA2)
Other:
- note added: "I2C"
- note added: "SPI"
- note added: "UART"

Commit message: Write project specification
Parts:
- R: renamed from R?; value R -> 10k
- R: renamed from R?; value R -> 4k
Other:
- title: (none) -> Měření vzdálenosti na základě vířivých proudů
- moved on the sheet: R
Changed lines of the file:
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@@
 (kicad_sch (version 20211123) (generator eeschema)
   (paper "A4")
+  (title_block
+    (title "Měření vzdálenosti na základě vířivých proudů")
+    (date "2022-12-01")
+  )
   (junction (at 214.63 116.84) (diameter 0) (color 0 0 0 0)
   )
@@
     (stroke (width 0) (type default) (color 0 0 0 0))
   )
-  (wire (pts (xy 233.68 101.6) (xy 242.57 101.6))
+  (wire (pts (xy 241.3 101.6) (xy 242.57 101.6))
     (stroke (width 0) (type default) (color 0 0 0 0))
   )
@@
     (stroke (width 0) (type default) (color 0 0 0 0))
   )
-  (wire (pts (xy 218.44 101.6) (xy 226.06 101.6))
+  (wire (pts (xy 218.44 101.6) (xy 233.68 101.6))
     (stroke (width 0) (type default) (color 0 0 0 0))
   )
@@
   (symbol (lib_id "Device:R") (at 200.66 96.52 0) (unit 1)
     (in_bom yes) (on_board yes) (fields_autoplaced)
-    (property "Reference" "R?" (id 0) (at 203.2 95.2499 0)
+    (property "Reference" "R" (id 0) (at 203.2 95.2499 0)
       (effects (font (size 1.27 1.27)) (justify left))
     )
-    (property "Value" "R" (id 1) (at 203.2 97.7899 0)
+    (property "Value" "10k" (id 1) (at 203.2 97.7899 0)
       (effects (font (size 1.27 1.27)) (justify left))
     )
@@
     (pin "2")
   )
-  (symbol (lib_id "Device:R") (at 229.87 101.6 90) (unit 1)
-    (in_bom yes) (on_board yes) (fields_autoplaced)
-    (property "Reference" "R?" (id 0) (at 229.87 95.25 90))
-    (property "Value" "R" (id 1) (at 229.87 97.79 90))
-    (property "Footprint" "" (id 2) (at 229.87 103.378 90)
-      (effects (font (size 1.27 1.27)) hide)
-    )
-    (property "Datasheet" "~" (id 3) (at 229.87 101.6 0)
+  (symbol (lib_id "Device:R") (at 237.49 101.6 90) (mirror x) (unit 1)
+    (in_bom yes) (on_board yes) (fields_autoplaced)
+    (property "Reference" "R" (id 0) (at 237.49 95.25 90))
+    (property "Value" "4k" (id 1) (at 237.49 97.79 90))
+    (property "Footprint" "" (id 2) (at 237.49 99.822 90)
+      (effects (font (size 1.27 1.27)) hide)
+    )
+    (property "Datasheet" "~" (id 3) (at 237.49 101.6 0)
       (effects (font (size 1.27 1.27)) hide)
     )
@@
   (symbol (lib_id "Device:R") (at 218.44 107.95 0) (unit 1)
     (in_bom yes) (on_board yes) (fields_autoplaced)
-    (property "Reference" "R?" (id 0) (at 220.98 106.6799 0)
+    (property "Reference" "R" (id 0) (at 220.98 106.6799 0)
       (effects (font (size 1.27 1.27)) (justify left))
     )
-    (property "Value" "R" (id 1) (at 220.98 109.2199 0)
+    (property "Value" "10k" (id 1) (at 220.98 109.2199 0)
       (effects (font (size 1.27 1.27)) (justify left))
     )
@@
     )
     (path "/0457ee33-48b2-4e84-9355-b3b18287742a"
-      (reference "R?") (unit 1) (value "R") (footprint "")
+      (reference "R") (unit 1) (value "10k") (footprint "")
     )
     (path "/df0ddedf-b20e-4980-9077-ed848e00fb64"
-      (reference "R?") (unit 1) (value "R") (footprint "")
+      (reference "R") (unit 1) (value "4k") (footprint "")
     )
     (path "/f498459b-3aaf-4849-86eb-e72ecc3d9fa3"
-      (reference "R?") (unit 1) (value "R") (footprint "")
+      (reference "R") (unit 1) (value "10k") (footprint "")
     )
     (path "/4ad87429-9101-474c-b67c-67637fbd9950"

Commit message: Update a KiCad
Connections:
- net RX: now also U?.25 (PA2), U?.68 (PA9); no longer U?.26 (PA3)
- net TX: now also U?.26 (PA3), U?.39 (PA10); no longer U?.25 (PA2)
Changed lines of the file:
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@@
     (date "2022-12-01")
   )
+  (junction (at 73.66 91.44) (diameter 0) (color 0 0 0 0)
+  )
   (junction (at 214.63 116.84) (diameter 0) (color 0 0 0 0)
   )
@@
   (junction (at 242.57 91.44) (diameter 0) (color 0 0 0 0)
   )
+  (junction (at 76.2 88.9) (diameter 0) (color 0 0 0 0)
+  )
   (wire (pts (xy 91.44 93.98) (xy 50.8 93.98))
     (stroke (width 0) (type default) (color 0 0 0 0))
@@
     (stroke (width 0) (type default) (color 0 0 0 0))
   )
+  (wire (pts (xy 165.1 149.86) (xy 76.2 149.86))
+    (stroke (width 0) (type default) (color 0 0 0 0))
+  )
   (polyline (pts (xy 24.13 129.54) (xy 41.91 129.54))
     (stroke (width 0) (type default) (color 0 0 0 0))
@@
     (stroke (width 0) (type default) (color 0 0 0 0))
   )
+  (wire (pts (xy 76.2 88.9) (xy 91.44 88.9))
+    (stroke (width 0) (type default) (color 0 0 0 0))
+  )
+  (wire (pts (xy 162.56 99.06) (xy 140.97 99.06))
+    (stroke (width 0) (type default) (color 0 0 0 0))
+  )
+  (wire (pts (xy 162.56 99.06) (xy 162.56 152.4))
+    (stroke (width 0) (type default) (color 0 0 0 0))
+  )
   (polyline (pts (xy 41.91 129.54) (xy 41.91 106.68))
     (stroke (width 0) (type default) (color 0 0 0 0))
@@
     (stroke (width 0) (type default) (color 0 0 0 0))
   )
+  (wire (pts (xy 73.66 152.4) (xy 73.66 91.44))
+    (stroke (width 0) (type default) (color 0 0 0 0))
+  )
   (wire (pts (xy 91.44 73.66) (xy 55.88 73.66))
     (stroke (width 0) (type default) (color 0 0 0 0))
@@
     (stroke (width 0) (type default) (color 0 0 0 0))
   )
+  (wire (pts (xy 165.1 101.6) (xy 165.1 149.86))
+    (stroke (width 0) (type default) (color 0 0 0 0))
+  )
   (wire (pts (xy 53.34 96.52) (xy 53.34 115.57))
     (stroke (width 0) (type default) (color 0 0 0 0))
@@
     (stroke (width 0) (type default) (color 0 0 0 0))
   )
-  (wire (pts (xy 36.83 91.44) (xy 91.44 91.44))
+  (wire (pts (xy 36.83 91.44) (xy 73.66 91.44))
+    (stroke (width 0) (type default) (color 0 0 0 0))
+  )
+  (wire (pts (xy 162.56 152.4) (xy 73.66 152.4))
     (stroke (width 0) (type default) (color 0 0 0 0))
   )
@@
     (stroke (width 0) (type default) (color 0 0 0 0))
   )
+  (wire (pts (xy 73.66 91.44) (xy 91.44 91.44))
+    (stroke (width 0) (type default) (color 0 0 0 0))
+  )
   (wire (pts (xy 218.44 101.6) (xy 233.68 101.6))
     (stroke (width 0) (type default) (color 0 0 0 0))
@@
     (stroke (width 0.5) (type solid) (color 86 86 86 1))
   )
+  (wire (pts (xy 140.97 101.6) (xy 165.1 101.6))
+    (stroke (width 0) (type default) (color 0 0 0 0))
+  )
   (wire (pts (xy 222.25 93.98) (xy 218.44 93.98))
     (stroke (width 0) (type default) (color 0 0 0 0))
@@
     (stroke (width 0) (type default) (color 0 0 0 0))
   )
+  (wire (pts (xy 76.2 88.9) (xy 76.2 149.86))
+    (stroke (width 0) (type default) (color 0 0 0 0))
+  )
   (wire (pts (xy 242.57 91.44) (xy 251.46 91.44))
     (stroke (width 0) (type default) (color 0 0 0 0))
@@
     (stroke (width 0) (type default) (color 0 0 0 0))
   )
-  (wire (pts (xy 36.83 88.9) (xy 91.44 88.9))
+  (wire (pts (xy 36.83 88.9) (xy 76.2 88.9))
     (stroke (width 0) (type default) (color 0 0 0 0))
   )
@@
     (effects (font (size 3 3)) (justify left bottom))
   )
+  (label "USART1_RX" (at 143.51 99.06 0)
+    (effects (font (size 1.27 1.27)) (justify left bottom))
+  )
   (label "SPI1_SCK" (at 90.17 96.52 180)
     (effects (font (size 1.27 1.27)) (justify right bottom))
   )
-  (label "RX" (at 36.83 91.44 0)
+  (label "TX" (at 36.83 91.44 0)
     (effects (font (size 1.27 1.27)) (justify left bottom))
   )
@@
     (effects (font (size 1.27 1.27)) (justify right bottom))
   )
+  (label "USART1_TX" (at 143.51 101.6 0)
+    (effects (font (size 1.27 1.27)) (justify left bottom))
+  )
   (label "SPI1_MOSI" (at 80.01 101.6 0)
     (effects (font (size 1.27 1.27)) (justify left bottom))
@@
     (effects (font (size 1.27 1.27)) (justify left bottom))
   )
-  (label "TX" (at 36.83 88.9 0)
-    (effects (font (size 1.27 1.27)) (justify left bottom))
-  )
+  (label "RX" (at 36.83 88.9 0)
+    (effects (font (size 1.27 1.27)) (justify left bottom))
+  )

Commit message: Update a project shema
Parts:
- removed R: 4k, symbol Device:R
- removed R: 10k, symbol Device:R
- removed U?: Opamp_Dual, symbol Device:Opamp_Dual
Connections:
- net ADC1_IN10: now also L?.2, R.1
- net MISO: no longer names the net of U?.31 (PA6)
- net MOSI: no longer names the net of U?.32 (PA7)
- net NSS: no longer names the net of U?.29 (PA4)
- net SCK: no longer names the net of U?.30 (PA5)
Other:
- note removed: "SPI"
